File: 60Keyboard.kicad_pcb (KiCad board)
At the start: 2 copper layers, 134 parts

Commit message: updated edge cut & manufacturing files
Parts:
- moved U1 0.46 mm to (294.7, 17.0)
Routing:
- net Column 4: track 323.1 -> 324.2 mm
- net Column 3: track 306.4 -> 307.0 mm
- added copper zone on B.Cu, net (none)
- added copper zone on F.Cu, net (none)
Other:
- board outline added: 307 x 96 mm
